File: kikad/Placa-Final/Placa-Final.kicad_pcb (KiCad board)
At the start: 2 copper layers, 100 x 100 mm, 32 parts, among them SW1 SW_Push, SW2 SW_Push, SW3 SW_Push, SW4 SW_Push, U1 ESP32-WROOM-32, U2 RS232, U3 MicroSDCardAdapter, U4 HW-504, U5 LM2596, U6 XL6009E1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

Commit message: Add files via upload
Parts:
- moved U7 31.2 mm to (82.5, 96.5), turned to -90 degrees
- moved C4 9.06 mm to (80.5, 108.7)
- moved R5 9.06 mm to (72.7, 113.2)
- moved C3 9.06 mm to (70.3, 108.7)
- moved R4 9.06 mm to (67.9, 113.2)
- moved R6 9.06 mm to (78.1, 113.1)
- moved SW3 9.06 mm to (67.8, 123.9)
- moved SW4 9.06 mm to (78.0, 123.9)
- moved R7 9.06 mm to (83.0, 113.1)
Routing:
- net +5V: track 171.9 -> 137.2 mm
- net GNDPWR: track 166.1 -> 136.0 mm
- net SCLi2c: track 79.6 -> 51.3 mm
- net SADi2c: track 79.2 -> 52.7 mm
- net +3V3: track 144.0 -> 159.4 mm
- net GND: track 180.2 -> 189.1 mm
- net SW: track 45.6 -> 52.1 mm
- net VRY: track 44.2 -> 48.9 mm
- net GNDREF: track 122.1 -> 119.2 mm
- net +4V: track 138.7 -> 137.6 mm

Commit message: Add files via upload
Routing:
- net +3V3: track 159.4 -> 165.4 mm
- net GND: track 189.1 -> 191.7 mm
- net +5V: track 137.2 -> 139.0 mm

Commit message: Add files via upload
Connections:
- D1 pad 1: GNDPWR -> GND
- U3 pad 1: GNDPWR -> GND
- U4 pad 1: GNDPWR -> GND
- U5 pad 2: GNDREF -> GND
- U6 pad 2: GNDREF -> GND
- U6 pad 4: GNDPWR -> GND
- U7 pad 1: GNDPWR -> GND
- U8 pad 6: GNDPWR -> GND
- U9 pad 4: GNDREF -> GND
Routing:
- net GND: track 191.7 -> 0.00 mm, vias 1 -> 0
- net GNDPWR: track 135.8 -> 0.00 mm
- net GNDREF: track 119.2 -> 0.00 mm
- net +3V3: track 165.4 -> 184.3 mm, vias 0 -> 3
- net +5V: track 139.0 -> 145.7 mm
- net B1: track 5.73 -> 0.00 mm
- net SW: track 52.1 -> 54.4 mm
- net VRY: track 48.9 -> 50.5 mm
- net Net-(SW1-Pad2): track 34.5 -> 35.9 mm
- added copper zone on B.Cu, net GND
- added copper zone on F.Cu, net GND

Commit message: Add files via upload
Parts:
- added ?: , , F.Cu at (82.2, 34.0)
- added ?: , , F.Cu at (34.0, 125.7)
- added ?: , , F.Cu at (125.6, 34.3)
- added ?: , , F.Cu at (81.8, 71.9)
- C1, C2, C3, C4: footprint Capacitor_SMD:C_1206_3216Metric_Pad1.33x1.80mm_HandSolder -> Capacitor_SMD:C_0805_2012Metric_Pad1.18x1.45mm_HandSolder
Routing:
- net +3V3: track 184.3 -> 190.6 mm, vias 3 -> 2
- net B1: track 0.00 -> 5.73 mm
- net +4V: track 138.0 -> 139.8 mm
- net +5V: track 145.7 -> 147.5 mm
- net Net-(BT1-Pad1): track 13.9 -> 15.3 mm
- net Net-(R7-Pad2): track 14.3 -> 15.0 mm
- net SCLi2c: track 51.3 -> 51.9 mm
- net VRY: track 50.5 -> 51.0 mm
- net Net-(R5-Pad2): track 14.2 -> 14.7 mm
- net GND: vias 0 -> 396
