File: kikad/Placa-Final/Placa-Final.kicad_sch (KiCad schematic)
At the start: 32 parts, among them SW1 SW_Push, SW2 SW_Push, SW3 SW_Push, SW4 SW_Push, U1 ESP32-WROOM-32, U2 RS232, U3 MicroSDCardAdapter, U4 HW-504, U5 LM2596, U6 XL6009E1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

Commit message: Add files via upload
Connections:
- net GNDPWR is gone; now on net GND: D1.1 (K), U3.1 (Gnd), U4.1 (GND), U6.4 (OUT-), U7.1 (GND), U8.6 (GND)
- net GNDREF is gone; now on net GND: U5.2 (IN-), U6.2 (IN-), U9.4 (Out-)

Commit message: Add files via upload
Parts:
- C1, C2, C3, C4: footprint Capacitor_SMD:C_1206_3216Metric_Pad1.33x1.80mm_HandSolder -> Capacitor_SMD:C_0805_2012Metric_Pad1.18x1.45mm_HandSolder
Changed lines of the file:
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@@
       (effects (font (size 1.27 1.27)) (justify right))
     )
-    (property "Footprint" "Capacitor_SMD:C_1206_3216Metric_Pad1.33x1.80mm_HandSolder" (id 2) (at 120.9548 63.5 0)
+    (property "Footprint" "Capacitor_SMD:C_0805_2012Metric_Pad1.18x1.45mm_HandSolder" (id 2) (at 120.9548 63.5 0)
       (effects (font (size 1.27 1.27)) hide)
     )
@@
     (property "Reference" "C1" (id 0) (at 26.67 49.53 90))
     (property "Value" "100n" (id 1) (at 26.67 52.07 90))
-    (property "Footprint" "Capacitor_SMD:C_1206_3216Metric_Pad1.33x1.80mm_HandSolder" (id 2) (at 30.48 56.1848 0)
+    (property "Footprint" "Capacitor_SMD:C_0805_2012Metric_Pad1.18x1.45mm_HandSolder" (id 2) (at 30.48 56.1848 0)
       (effects (font (size 1.27 1.27)) hide)
     )
@@
       (effects (font (size 1.27 1.27)) (justify right))
     )
-    (property "Footprint" "Capacitor_SMD:C_1206_3216Metric_Pad1.33x1.80mm_HandSolder" (id 2) (at 120.9548 114.3 0)
+    (property "Footprint" "Capacitor_SMD:C_0805_2012Metric_Pad1.18x1.45mm_HandSolder" (id 2) (at 120.9548 114.3 0)
       (effects (font (size 1.27 1.27)) hide)
     )
@@
   (symbol (lib_id "power:GND") (at 218.44 62.23 0) (unit 1)
     (in_bom yes) (on_board yes) (fields_autoplaced)
-    (property "Reference" "#PWR?" (id 0) (at 218.44 68.58 0)
+    (property "Reference" "#PWR0119" (id 0) (at 218.44 68.58 0)
       (effects (font (size 1.27 1.27)) hide)
     )
@@
     (property "Reference" "C2" (id 0) (at 77.47 49.53 90))
     (property "Value" "100n" (id 1) (at 77.47 52.07 90))
-    (property "Footprint" "Capacitor_SMD:C_1206_3216Metric_Pad1.33x1.80mm_HandSolder" (id 2) (at 81.28 56.1848 0)
+    (property "Footprint" "Capacitor_SMD:C_0805_2012Metric_Pad1.18x1.45mm_HandSolder" (id 2) (at 81.28 56.1848 0)
       (effects (font (size 1.27 1.27)) hide)
     )
@@
   (symbol (lib_id "power:GND") (at 219.71 82.55 0) (unit 1)
     (in_bom yes) (on_board yes) (fields_autoplaced)
-    (property "Reference" "#PWR?" (id 0) (at 219.71 88.9 0)
+    (property "Reference" "#PWR0104" (id 0) (at 219.71 88.9 0)
       (effects (font (size 1.27 1.27)) hide)
     )
@@
       (reference "#PWR0103") (unit 1) (value "+4V") (footprint "")
     )
+    (path "/f2b6e32b-edf2-4804-861b-99e72f72470c"
+      (reference "#PWR0104") (unit 1) (value "GND") (footprint "")
+    )
     (path "/1d8298f6-5278-42d3-9c9d-3fd92e9421e2"
       (reference "#PWR0105") (unit 1) (value "+4V") (footprint "")
@@
       (reference "#PWR0118") (unit 1) (value "+4V") (footprint "")
     )
+    (path "/dc494e81-b50b-453c-ba8e-8cfe2ab07aab"
+      (reference "#PWR0119") (unit 1) (value "GND") (footprint "")
+    )
     (path "/bfb9a383-1f8c-4547-81c9-2c710f5dc4f6"
       (reference "#PWR0120") (unit 1) (value "GND") (footprint "")
@@
       (reference "#PWR0128") (unit 1) (value "+3.3V") (footprint "")
     )
-    (path "/dc494e81-b50b-453c-ba8e-8cfe2ab07aab"
-      (reference "#PWR?") (unit 1) (value "GND") (footprint "")
-    )
-    (path "/f2b6e32b-edf2-4804-861b-99e72f72470c"
-      (reference "#PWR?") (unit 1) (value "GND") (footprint "")
-    )
     (path "/78d2299b-0fcd-4ea5-ba66-3ab5aaf4d0b5"
       (reference "BT1") (unit 1) (value "Battery_Cell") (footprint "Connector_PinHeader_2.54mm:PinHeader_1x02_P2.54mm_Vertical")
     )
     (path "/6926fa33-b483-4b27-9021-c8c173bee123"
-      (reference "C1") (unit 1) (value "100n") (footprint "Capacitor_SMD:C_1206_3216Metric_Pad1.33x1.80mm_HandSolder")
+      (reference "C1") (unit 1) (value "100n") (footprint "Capacitor_SMD:C_0805_2012Metric_Pad1.18x1.45mm_HandSolder")
     )
     (path "/e4e67376-2997-4cd7-8772-d58858687656"
-      (reference "C2") (unit 1) (value "100n") (footprint "Capacitor_SMD:C_1206_3216Metric_Pad1.33x1.80mm_HandSolder")
+      (reference "C2") (unit 1) (value "100n") (footprint "Capacitor_SMD:C_0805_2012Metric_Pad1.18x1.45mm_HandSolder")
     )
     (path "/58f6bfb6-8660-4af0-9f62-3d217f193d18"
-      (reference "C3") (unit 1) (value "100n") (footprint "Capacitor_SMD:C_1206_3216Metric_Pad1.33x1.80mm_HandSolder")
+      (reference "C3") (unit 1) (value "100n") (footprint "Capacitor_SMD:C_0805_2012Metric_Pad1.18x1.45mm_HandSolder")
     )
     (path "/ca116935-d445-4a5c-9020-376614502193"
-      (reference "C4") (unit 1) (value "100n") (footprint "Capacitor_SMD:C_1206_3216Metric_Pad1.33x1.80mm_HandSolder")
+      (reference "C4") (unit 1) (value "100n") (footprint "Capacitor_SMD:C_0805_2012Metric_Pad1.18x1.45mm_HandSolder")
     )
     (path "/f0913a11-bf78-4ce7-8e04-139da3800ce3"
